File: DCDC_Converter_DemoBoard.kicad_pcb (KiCad board)
At the start: 2 copper layers, 183 x 38 mm, 82 parts, among them J1 Conn_01x01, J10 Conn_01x01, J11 Conn_01x01, J12 Conn_01x01, J13 Conn_01x01, J14 Conn_01x01, J15 Conn_01x01, J16 Conn_01x01, J2 Conn_01x01, J3 Conn_01x01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

Commit message: fixed footprint and cleaned up silkscreen
Parts:
- L15, L16: footprint Inductor_SMD:L_1008_2520Metric_Pad1.43x2.20mm_HandSolder -> Inductor_SMD:L_1812_4532Metric_Pad1.30x3.40mm_HandSolder
Routing:
- net Net-(JP23-B): track 3.90 -> 6.36 mm
- net Net-(JP26-B): track 7.24 -> 6.17 mm
- net Net-(JP24-B): track 7.46 -> 6.40 mm
- net GND: vias 486 -> 485
